Commit message: update urdf

File: RIVO_description/urdf/RIVO.xacro (robot description, xacro)
@@ -4,7 +4,14 @@
 <xacro:include filename="$(find RIVO_description)/urdf/RIVO.trans" />
 <xacro:include filename="$(find RIVO_description)/urdf/RIVO.gazebo" />
+<link name="dummy_link">
+  <pose>0 0 0 0 0 0</pose>
+</link>
+<joint name="dummy_joint" type="fixed">
+  <parent link="dummy_link"/>
+  <child link="base_link"/>
+</joint>
 <link name="base_link">
   <inertial>
-    <origin xyz="0.0028948644801508917 0.0004061893631920199 -0.06237868835414986" rpy="0 0 0"/>
+    <origin xyz="0.002894864480150963 0.0004061893631920555 0.029121311645850093" rpy="0 0 0"/>
     <mass value="2.3408931898157137"/>
     <inertia ixx="0.004521" iyy="0.004886" izz="0.00607" ixy="4e-06" iyz="-9e-06" ixz="5.9e-05"/>
@@ -26,10 +33,10 @@
 <link name="link_2_1">
   <inertial>
-    <origin xyz="0.0020835623132613285 -0.003064482171297948 0.019940090429391336" rpy="0 0 0"/>
+    <origin xyz="0.002083562313261399 -0.003064482171298019 0.019940090429391252" rpy="0 0 0"/>
     <mass value="0.688307702528786"/>
     <inertia ixx="0.000549" iyy="0.000566" izz="0.000619" ixy="6e-06" iyz="1.3e-05" ixz="-6.5e-05"/>
   </inertial>
   <visual>
-    <origin xyz="3.5e-05 -1.6e-05 2e-06" rpy="0 0 0"/>
+    <origin xyz="3.5e-05 -1.6e-05 -0.091498" rpy="0 0 0"/>
     <geometry>
       <mesh filename="package://RIVO_description/meshes/link_2_1.stl" scale="0.001 0.001 0.001"/>
@@ -38,5 +45,5 @@
   </visual>
   <collision>
-    <origin xyz="3.5e-05 -1.6e-05 2e-06" rpy="0 0 0"/>
+    <origin xyz="3.5e-05 -1.6e-05 -0.091498" rpy="0 0 0"/>
     <geometry>
       <mesh filename="package://RIVO_description/meshes/link_2_1.stl" scale="0.001 0.001 0.001"/>
@@ -46,10 +53,10 @@
 <link name="link_4_1">
   <inertial>
-    <origin xyz="0.08125834087790981 -0.001122555428102228 0.00029418621949284934" rpy="0 0 0"/>
+    <origin xyz="0.08125834087790981 -0.001122555428102228 0.0002941862194928979" rpy="0 0 0"/>
     <mass value="0.46578916720940555"/>
     <inertia ixx="6.1e-05" iyy="0.001753" izz="0.001704" ixy="-4.8e-05" iyz="-0.0" ixz="-1.2e-05"/>
   </inertial>
   <visual>
-    <origin xyz="-0.231507 0.019199 -0.039643" rpy="0 0 0"/>
+    <origin xyz="-0.231507 0.019199 -0.131143" rpy="0 0 0"/>
     <geometry>
       <mesh filename="package://RIVO_description/meshes/link_4_1.stl" scale="0.001 0.001 0.001"/>
@@ -58,5 +65,5 @@
   </visual>
   <collision>
-    <origin xyz="-0.231507 0.019199 -0.039643" rpy="0 0 0"/>
+    <origin xyz="-0.231507 0.019199 -0.131143" rpy="0 0 0"/>
     <geometry>
       <mesh filename="package://RIVO_description/meshes/link_4_1.stl" scale="0.001 0.001 0.001"/>
@@ -64,221 +71,221 @@
   </collision>
 </link>
-<link name="gripper_part_12_1">
-  <inertial>
-    <origin xyz="0.012456635259577353 0.009213868537273885 0.0020449037369226486" rpy="0 0 0"/>
+<link name="g_part_12_1">
+  <inertial>
+    <origin xyz="0.012456635259577353 0.009213868537273885 0.0020449037369225376" rpy="0 0 0"/>
     <mass value="0.006270284943512531"/>
     <inertia ixx="0.0" iyy="1e-06" izz="1e-06" ixy="-0.0" iyz="-0.0" ixz="-0.0"/>
   </inertial>
   <visual>
-    <origin xyz="-0.484567 -0.00431 -0.055238" rpy="0 0 0"/>
-    <geometry>
-      <mesh filename="package://RIVO_description/meshes/gripper_part_12_1.stl" scale="0.001 0.001 0.001"/>
-    </geometry>
-    <material name="silver"/>
-  </visual>
-  <collision>
-    <origin xyz="-0.484567 -0.00431 -0.055238" rpy="0 0 0"/>
-    <geometry>
-      <mesh filename="package://RIVO_description/meshes/gripper_part_12_1.stl" scale="0.001 0.001 0.001"/>
-    </geometry>
-  </collision>
-</link>
-<link name="gripper_part_4_1">
-  <inertial>
-    <origin xyz="0.013134263289696746 -0.008251164752194744 0.0019147897203106931" rpy="0 0 0"/>
+    <origin xyz="-0.484567 -0.00431 -0.146738" rpy="0 0 0"/>
+    <geometry>
+      <mesh filename="package://RIVO_description/meshes/g_part_12_1.stl" scale="0.001 0.001 0.001"/>
+    </geometry>
+    <material name="silver"/>
+  </visual>
+  <collision>
+    <origin xyz="-0.484567 -0.00431 -0.146738" rpy="0 0 0"/>
+    <geometry>
+      <mesh filename="package://RIVO_description/meshes/g_part_12_1.stl" scale="0.001 0.001 0.001"/>
+    </geometry>
+  </collision>
+</link>
+<link name="g_part_4_1">
+  <inertial>
+    <origin xyz="0.013134263289696746 -0.008251164752194753 0.0019147897203106445" rpy="0 0 0"/>
     <mass value="0.006270284943499826"/>
     <inertia ixx="0.0" iyy="1e-06" izz="1e-06" ixy="0.0" iyz="-0.0" ixz="0.0"/>
   </inertial>
   <visual>
-    <origin xyz="-0.484828 0.005686 -0.055163" rpy="0 0 0"/>
-    <geometry>
-      <mesh filename="package://RIVO_description/meshes/gripper_part_4_1.stl" scale="0.001 0.001 0.001"/>
-    </geometry>
-    <material name="silver"/>
-  </visual>
-  <collision>
-    <origin xyz="-0.484828 0.005686 -0.055163" rpy="0 0 0"/>
-    <geometry>
-      <mesh filename="package://RIVO_description/meshes/gripper_part_4_1.stl" scale="0.001 0.001 0.001"/>
-    </geometry>
-  </collision>
-</link>
-<link name="gripper_part_8_1">
-  <inertial>
-    <origin xyz="0.0105618667457274 0.007870370761826763 -0.004894936320047574" rpy="0 0 0"/>
+    <origin xyz="-0.484828 0.005686 -0.146663" rpy="0 0 0"/>
+    <geometry>
+      <mesh filename="package://RIVO_description/meshes/g_part_4_1.stl" scale="0.001 0.001 0.001"/>
+    </geometry>
+    <material name="silver"/>
+  </visual>
+  <collision>
+    <origin xyz="-0.484828 0.005686 -0.146663" rpy="0 0 0"/>
+    <geometry>
+      <mesh filename="package://RIVO_description/meshes/g_part_4_1.stl" scale="0.001 0.001 0.001"/>
+    </geometry>
+  </collision>
+</link>
+<link name="g_part_8_1">
+  <inertial>
+    <origin xyz="0.0105618667457274 0.00787037076182677 -0.004894936320047616" rpy="0 0 0"/>
     <mass value="0.007386988595910961"/>
     <inertia ixx="0.0" iyy="1e-06" izz="1e-06" ixy="-0.0" iyz="0.0" ixz="0.0"/>
   </inertial>
   <visual>
-    <origin xyz="-0.484556 -0.004351 -0.049669" rpy="0 0 0"/>
-    <geometry>
-      <mesh filename="package://RIVO_description/meshes/gripper_part_8_1.stl" scale="0.001 0.001 0.001"/>
-    </geometry>
-    <material name="silver"/>
-  </visual>
-  <collision>
-    <origin xyz="-0.484556 -0.004351 -0.049669" rpy="0 0 0"/>
-    <geometry>
-      <mesh filename="package://RIVO_description/meshes/gripper_part_8_1.stl" scale="0.001 0.001 0.001"/>
-    </geometry>
-  </collision>
-</link>
-<link name="gripper_part_2_1">
-  <inertial>
-    <origin xyz="-0.00036726587359098284 0.01348177608821506 -0.008550972042145076" rpy="0 0 0"/>
+    <origin xyz="-0.484556 -0.004351 -0.141169" rpy="0 0 0"/>
+    <geometry>
+      <mesh filename="package://RIVO_description/meshes/g_part_8_1.stl" scale="0.001 0.001 0.001"/>
+    </geometry>
+    <material name="silver"/>
+  </visual>
+  <collision>
+    <origin xyz="-0.484556 -0.004351 -0.141169" rpy="0 0 0"/>
+    <geometry>
+      <mesh filename="package://RIVO_description/meshes/g_part_8_1.stl" scale="0.001 0.001 0.001"/>
+    </geometry>
+  </collision>
+</link>
+<link name="g_part_2_1">
+  <inertial>
+    <origin xyz="-0.00036726587359098284 0.01348177608821506 -0.00855097204214511" rpy="0 0 0"/>
     <mass value="0.05700410540308347"/>
     <inertia ixx="6e-06" iyy="4e-06" izz="3e-06" ixy="0.0" iyz="0.0" ixz="-0.0"/>
   </inertial>
   <visual>
-    <origin xyz="-0.464814 0.006035 -0.045128" rpy="0 0 0"/>
-    <geometry>
-      <mesh filename="package://RIVO_description/meshes/gripper_part_2_1.stl" scale="0.001 0.001 0.001"/>
-    </geometry>
-    <material name="silver"/>
-  </visual>
-  <collision>
-    <origin xyz="-0.464814 0.006035 -0.045128" rpy="0 0 0"/>
-    <geometry>
-      <mesh filename="package://RIVO_description/meshes/gripper_part_2_1.stl" scale="0.001 0.001 0.001"/>
-    </geometry>
-  </collision>
-</link>
-<link name="gripper_part_9_1">
-  <inertial>
-    <origin xyz="0.005021384222760938 -0.0025433255854703136 0.003471513807427669" rpy="0 0 0"/>
+    <origin xyz="-0.464814 0.006035 -0.136628" rpy="0 0 0"/>
+    <geometry>
+      <mesh filename="package://RIVO_description/meshes/g_part_2_1.stl" scale="0.001 0.001 0.001"/>
+    </geometry>
+    <material name="silver"/>
+  </visual>
+  <collision>
+    <origin xyz="-0.464814 0.006035 -0.136628" rpy="0 0 0"/>
+    <geometry>
+      <mesh filename="package://RIVO_description/meshes/g_part_2_1.stl" scale="0.001 0.001 0.001"/>
+    </geometry>
+  </collision>
+</link>
+<link name="g_part_9_1">
+  <inertial>
+    <origin xyz="0.005021384222760994 -0.0025433255854703206 0.0034715138074274954" rpy="0 0 0"/>
     <mass value="0.0362891624976011"/>
     <inertia ixx="3e-06" iyy="4e-06" izz="6e-06" ixy="2e-06" iyz="-0.0" ixz="0.0"/>
   </inertial>
   <visual>
-    <origin xyz="-0.465043 0.014202 -0.054568" rpy="0 0 0"/>
-    <geometry>
-      <mesh filename="package://RIVO_description/meshes/gripper_part_9_1.stl" scale="0.001 0.001 0.001"/>
-    </geometry>
-    <material name="silver"/>
-  </visual>
-  <collision>
-    <origin xyz="-0.465043 0.014202 -0.054568" rpy="0 0 0"/>
-    <geometry>
-      <mesh filename="package://RIVO_description/meshes/gripper_part_9_1.stl" scale="0.001 0.001 0.001"/>
-    </geometry>
-  </collision>
-</link>
-<link name="gripper_part_10_1">
-  <inertial>
-    <origin xyz="-0.014598965910585904 0.008272324580325768 8.800201478370573e-05" rpy="0 0 0"/>
+    <origin xyz="-0.465043 0.014202 -0.146068" rpy="0 0 0"/>
+    <geometry>
+      <mesh filename="package://RIVO_description/meshes/g_part_9_1.stl" scale="0.001 0.001 0.001"/>
+    </geometry>
+    <material name="silver"/>
+  </visual>
+  <collision>
+    <origin xyz="-0.465043 0.014202 -0.146068" rpy="0 0 0"/>
+    <geometry>
+      <mesh filename="package://RIVO_description/meshes/g_part_9_1.stl" scale="0.001 0.001 0.001"/>
+    </geometry>
+  </collision>
+</link>
+<link name="g_part_10_1">
+  <inertial>
+    <origin xyz="-0.014598965910585904 0.008272324580325768 8.800201478362246e-05" rpy="0 0 0"/>
     <mass value="0.05700410540308428"/>
     <inertia ixx="4e-06" iyy="3e-06" izz="6e-06" ixy="-0.0" iyz="-0.0" ixz="0.0"/>
   </inertial>
   <visual>
-    <origin xyz="-0.444042 0.006395 -0.040664" rpy="0 0 0"/>
-    <geometry>
-      <mesh filename="package://RIVO_description/meshes/gripper_part_10_1.stl" scale="0.001 0.001 0.001"/>
-    </geometry>
-    <material name="silver"/>
-  </visual>
-  <collision>
-    <origin xyz="-0.444042 0.006395 -0.040664" rpy="0 0 0"/>
-    <geometry>
-      <mesh filename="package://RIVO_description/meshes/gripper_part_10_1.stl" scale="0.001 0.001 0.001"/>
-    </geometry>
-  </collision>
-</link>
-<link name="gripper_part_1_1">
-  <inertial>
-    <origin xyz="0.036423386056162965 0.011494519998513543 0.006746851708180859" rpy="0 0 0"/>
+    <origin xyz="-0.444042 0.006395 -0.132164" rpy="0 0 0"/>
+    <geometry>
+      <mesh filename="package://RIVO_description/meshes/g_part_10_1.stl" scale="0.001 0.001 0.001"/>
+    </geometry>
+    <material name="silver"/>
+  </visual>
+  <collision>
+    <origin xyz="-0.444042 0.006395 -0.132164" rpy="0 0 0"/>
+    <geometry>
+      <mesh filename="package://RIVO_description/meshes/g_part_10_1.stl" scale="0.001 0.001 0.001"/>
+    </geometry>
+  </collision>
+</link>
+<link name="g_part_1_1">
+  <inertial>
+    <origin xyz="0.036423386056162965 0.01149451999851355 0.006746851708180762" rpy="0 0 0"/>
     <mass value="0.1054118615130382"/>
     <inertia ixx="1.9e-05" iyy="4.8e-05" izz="5.5e-05" ixy="-1e-05" iyz="-3e-06" ixz="-9e-06"/>
   </inertial>
   <visual>
-    <origin xyz="-0.416441 0.014369 -0.040656" rpy="0 0 0"/>
-    <geometry>
-      <mesh filename="package://RIVO_description/meshes/gripper_part_1_1.stl" scale="0.001 0.001 0.001"/>
-    </geometry>
-    <material name="silver"/>
-  </visual>
-  <collision>
-    <origin xyz="-0.416441 0.014369 -0.040656" rpy="0 0 0"/>
-    <geometry>
-      <mesh filename="package://RIVO_description/meshes/gripper_part_1_1.stl" scale="0.001 0.001 0.001"/>
-    </geometry>
-  </collision>
-</link>
-<link name="gripper_part_6_1">
-  <inertial>
-    <origin xyz="0.010217406066357015 -0.0017233499857305587 0.004218909480987874" rpy="0 0 0"/>
+    <origin xyz="-0.416441 0.014369 -0.132156" rpy="0 0 0"/>
+    <geometry>
+      <mesh filename="package://RIVO_description/meshes/g_part_1_1.stl" scale="0.001 0.001 0.001"/>
+    </geometry>
+    <material name="silver"/>
+  </visual>
+  <collision>
+    <origin xyz="-0.416441 0.014369 -0.132156" rpy="0 0 0"/>
+    <geometry>
+      <mesh filename="package://RIVO_description/meshes/g_part_1_1.stl" scale="0.001 0.001 0.001"/>
+    </geometry>
+  </collision>
+</link>
+<link name="g_part_6_1">
+  <inertial>
+    <origin xyz="0.010217406066357015 -0.0017233499857305518 0.004218909480987715" rpy="0 0 0"/>
     <mass value="0.04741956072106952"/>
     <inertia ixx="1e-06" iyy="1.9e-05" izz="2e-05" ixy="-3e-06" iyz="0.0" ixz="0.0"/>
   </inertial>
   <visual>
-    <origin xyz="-0.511072 0.022091 -0.045923" rpy="0 0 0"/>
-    <geometry>
-      <mesh filename="package://RIVO_description/meshes/gripper_part_6_1.stl" scale="0.001 0.001 0.001"/>
-    </geometry>
-    <material name="silver"/>
-  </visual>
-  <collision>
-    <origin xyz="-0.511072 0.022091 -0.045923" rpy="0 0 0"/>
-    <geometry>
-      <mesh filename="package://RIVO_description/meshes/gripper_part_6_1.stl" scale="0.001 0.001 0.001"/>
-    </geometry>
-  </collision>
-</link>
-<link name="gripper_part_7_1">
-  <inertial>
-    <origin xyz="0.011136128559519176 -0.00695448952174929 -0.005005307666391845" rpy="0 0 0"/>
+    <origin xyz="-0.511072 0.022091 -0.137423" rpy="0 0 0"/>
+    <geometry>
+      <mesh filename="package://RIVO_description/meshes/g_part_6_1.stl" scale="0.001 0.001 0.001"/>
+    </geometry>
+    <material name="silver"/>
+  </visual>
+  <collision>
+    <origin xyz="-0.511072 0.022091 -0.137423" rpy="0 0 0"/>
+    <geometry>
+      <mesh filename="package://RIVO_description/meshes/g_part_6_1.stl" scale="0.001 0.001 0.001"/>
+    </geometry>
+  </collision>
+</link>
+<link name="g_part_7_1">
+  <inertial>
+    <origin xyz="0.011136128559519232 -0.006954489521749285 -0.005005307666391873" rpy="0 0 0"/>
     <mass value="0.007386988595910908"/>
     <inertia ixx="0.0" iyy="1e-06" izz="1e-06" ixy="0.0" iyz="-0.0" ixz="0.0"/>
   </inertial>
   <visual>
-    <origin xyz="-0.484818 0.005645 -0.049594" rpy="0 0 0"/>
-    <geometry>
-      <mesh filename="package://RIVO_description/meshes/gripper_part_7_1.stl" scale="0.001 0.001 0.001"/>
-    </geometry>
-    <material name="silver"/>
-  </visual>
-  <collision>
-    <origin xyz="-0.484818 0.005645 -0.049594" rpy="0 0 0"/>
-    <geometry>
-      <mesh filename="package://RIVO_description/meshes/gripper_part_7_1.stl" scale="0.001 0.001 0.001"/>
-    </geometry>
-  </collision>
-</link>
-<link name="gripper_part_3_1">
-  <inertial>
-    <origin xyz="-0.01973607073111644 -0.01515006847613012 0.0025168446301002192" rpy="0 0 0"/>
+    <origin xyz="-0.484818 0.005645 -0.141094" rpy="0 0 0"/>
+    <geometry>
+      <mesh filename="package://RIVO_description/meshes/g_part_7_1.stl" scale="0.001 0.001 0.001"/>
+    </geometry>
+    <material name="silver"/>
+  </visual>
+  <collision>
+    <origin xyz="-0.484818 0.005645 -0.141094" rpy="0 0 0"/>
+    <geometry>
+      <mesh filename="package://RIVO_description/meshes/g_part_7_1.stl" scale="0.001 0.001 0.001"/>
+    </geometry>
+  </collision>
+</link>
+<link name="g_part_3_1">
+  <inertial>
+    <origin xyz="-0.01973607073111644 -0.01515006847613011 0.002516844630100129" rpy="0 0 0"/>
     <mass value="0.02397572621792568"/>
     <inertia ixx="2e-06" iyy="2e-06" izz="4e-06" ixy="-1e-06" iyz="-0.0" ixz="0.0"/>
   </inertial>
   <visual>
-    <origin xyz="-0.489201 -0.031312 -0.055429" rpy="0 0 0"/>
-    <geometry>
-      <mesh filename="package://RIVO_description/meshes/gripper_part_3_1.stl" scale="0.001 0.001 0.001"/>
-    </geometry>
-    <material name="silver"/>
-  </visual>
-  <collision>
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