Commit message: update code

File: RIVO_description/urdf/RIVO.xacro (robot description, xacro)
@@ -1,427 +1,431 @@
 <?xml version="1.0" ?>
 <robot name="RIVO" xmlns:xacro="http://www.ros.org/wiki/xacro">
-<xacro:include filename="$(find RIVO_description)/urdf/materials.xacro" />
-<xacro:include filename="$(find RIVO_description)/urdf/RIVO.trans" />
-<xacro:include filename="$(find RIVO_description)/urdf/RIVO.gazebo" />
-<link name="dummy_link">
-  <pose>0 0 0 0 0 0</pose>
-</link>
-<joint name="dummy_joint" type="fixed">
-  <parent link="dummy_link"/>
-  <child link="base_link"/>
-</joint>
-<link name="base_link">
-  <inertial>
-    <origin xyz="0.002894864480150963 0.0004061893631920555 0.029121311645850093" rpy="0 0 0"/>
-    <mass value="2.3408931898157137"/>
-    <inertia ixx="0.004521" iyy="0.004886" izz="0.00607" ixy="4e-06" iyz="-9e-06" ixz="5.9e-05"/>
-  </inertial>
-  <visual>
-    <origin xyz="0 0 0" rpy="0 0 0"/>
-    <geometry>
-      <mesh filename="package://RIVO_description/meshes/base_link.stl" scale="0.001 0.001 0.001"/>
-    </geometry>
-    <material name="silver"/>
-  </visual>
-  <collision>
-    <origin xyz="0 0 0" rpy="0 0 0"/>
-    <geometry>
-      <mesh filename="package://RIVO_description/meshes/base_link.stl" scale="0.001 0.001 0.001"/>
-    </geometry>
-  </collision>
-</link>
-<link name="link_2_1">
-  <inertial>
-    <origin xyz="0.002083562313261399 -0.003064482171298019 0.019940090429391252" rpy="0 0 0"/>
-    <mass value="0.688307702528786"/>
-    <inertia ixx="0.000549" iyy="0.000566" izz="0.000619" ixy="6e-06" iyz="1.3e-05" ixz="-6.5e-05"/>
-  </inertial>
-  <visual>
-    <origin xyz="3.5e-05 -1.6e-05 -0.091498" rpy="0 0 0"/>
-    <geometry>
-      <mesh filename="package://RIVO_description/meshes/link_2_1.stl" scale="0.001 0.001 0.001"/>
-    </geometry>
-    <material name="silver"/>
-  </visual>
-  <collision>
-    <origin xyz="3.5e-05 -1.6e-05 -0.091498" rpy="0 0 0"/>
-    <geometry>
-      <mesh filename="package://RIVO_description/meshes/link_2_1.stl" scale="0.001 0.001 0.001"/>
-    </geometry>
-  </collision>
-</link>
-<link name="link_4_1">
-  <inertial>
-    <origin xyz="0.08125834087790981 -0.001122555428102228 0.0002941862194928979" rpy="0 0 0"/>
-    <mass value="0.46578916720940555"/>
-    <inertia ixx="6.1e-05" iyy="0.001753" izz="0.001704" ixy="-4.8e-05" iyz="-0.0" ixz="-1.2e-05"/>
-  </inertial>
-  <visual>
-    <origin xyz="-0.231507 0.019199 -0.131143" rpy="0 0 0"/>
-    <geometry>
-      <mesh filename="package://RIVO_description/meshes/link_4_1.stl" scale="0.001 0.001 0.001"/>
-    </geometry>
-    <material name="silver"/>
-  </visual>
-  <collision>
-    <origin xyz="-0.231507 0.019199 -0.131143" rpy="0 0 0"/>
-    <geometry>
-      <mesh filename="package://RIVO_description/meshes/link_4_1.stl" scale="0.001 0.001 0.001"/>
-    </geometry>
-  </collision>
-</link>
-<link name="g_part_12_1">
-  <inertial>
-    <origin xyz="0.012456635259577353 0.009213868537273885 0.0020449037369225376" rpy="0 0 0"/>
-    <mass value="0.006270284943512531"/>
-    <inertia ixx="0.0" iyy="1e-06" izz="1e-06" ixy="-0.0" iyz="-0.0" ixz="-0.0"/>
-  </inertial>
-  <visual>
-    <origin xyz="-0.484567 -0.00431 -0.146738" rpy="0 0 0"/>
-    <geometry>
-      <mesh filename="package://RIVO_description/meshes/g_part_12_1.stl" scale="0.001 0.001 0.001"/>
-    </geometry>
-    <material name="silver"/>
-  </visual>
-  <collision>
-    <origin xyz="-0.484567 -0.00431 -0.146738" rpy="0 0 0"/>
-    <geometry>
-      <mesh filename="package://RIVO_description/meshes/g_part_12_1.stl" scale="0.001 0.001 0.001"/>
-    </geometry>
-  </collision>
-</link>
-<link name="g_part_4_1">
-  <inertial>
-    <origin xyz="0.013134263289696746 -0.008251164752194753 0.0019147897203106445" rpy="0 0 0"/>
-    <mass value="0.006270284943499826"/>
-    <inertia ixx="0.0" iyy="1e-06" izz="1e-06" ixy="0.0" iyz="-0.0" ixz="0.0"/>
-  </inertial>
-  <visual>
-    <origin xyz="-0.484828 0.005686 -0.146663" rpy="0 0 0"/>
-    <geometry>
-      <mesh filename="package://RIVO_description/meshes/g_part_4_1.stl" scale="0.001 0.001 0.001"/>
-    </geometry>
-    <material name="silver"/>
-  </visual>
-  <collision>
-    <origin xyz="-0.484828 0.005686 -0.146663" rpy="0 0 0"/>
-    <geometry>
-      <mesh filename="package://RIVO_description/meshes/g_part_4_1.stl" scale="0.001 0.001 0.001"/>
-    </geometry>
-  </collision>
-</link>
-<link name="g_part_8_1">
-  <inertial>
-    <origin xyz="0.0105618667457274 0.00787037076182677 -0.004894936320047616" rpy="0 0 0"/>
-    <mass value="0.007386988595910961"/>
-    <inertia ixx="0.0" iyy="1e-06" izz="1e-06" ixy="-0.0" iyz="0.0" ixz="0.0"/>
-  </inertial>
-  <visual>
-    <origin xyz="-0.484556 -0.004351 -0.141169" rpy="0 0 0"/>
-    <geometry>
-      <mesh filename="package://RIVO_description/meshes/g_part_8_1.stl" scale="0.001 0.001 0.001"/>
-    </geometry>
-    <material name="silver"/>
-  </visual>
-  <collision>
-    <origin xyz="-0.484556 -0.004351 -0.141169" rpy="0 0 0"/>
-    <geometry>
-      <mesh filename="package://RIVO_description/meshes/g_part_8_1.stl" scale="0.001 0.001 0.001"/>
-    </geometry>
-  </collision>
-</link>
-<link name="g_part_2_1">
-  <inertial>
-    <origin xyz="-0.00036726587359098284 0.01348177608821506 -0.00855097204214511" rpy="0 0 0"/>
-    <mass value="0.05700410540308347"/>
-    <inertia ixx="6e-06" iyy="4e-06" izz="3e-06" ixy="0.0" iyz="0.0" ixz="-0.0"/>
-  </inertial>
-  <visual>
-    <origin xyz="-0.464814 0.006035 -0.136628" rpy="0 0 0"/>
-    <geometry>
-      <mesh filename="package://RIVO_description/meshes/g_part_2_1.stl" scale="0.001 0.001 0.001"/>
-    </geometry>
-    <material name="silver"/>
-  </visual>
-  <collision>
-    <origin xyz="-0.464814 0.006035 -0.136628" rpy="0 0 0"/>
-    <geometry>
-      <mesh filename="package://RIVO_description/meshes/g_part_2_1.stl" scale="0.001 0.001 0.001"/>
-    </geometry>
-  </collision>
-</link>
-<link name="g_part_9_1">
-  <inertial>
-    <origin xyz="0.005021384222760994 -0.0025433255854703206 0.0034715138074274954" rpy="0 0 0"/>
-    <mass value="0.0362891624976011"/>
-    <inertia ixx="3e-06" iyy="4e-06" izz="6e-06" ixy="2e-06" iyz="-0.0" ixz="0.0"/>
-  </inertial>
-  <visual>
-    <origin xyz="-0.465043 0.014202 -0.146068" rpy="0 0 0"/>
-    <geometry>
-      <mesh filename="package://RIVO_description/meshes/g_part_9_1.stl" scale="0.001 0.001 0.001"/>
-    </geometry>
-    <material name="silver"/>
-  </visual>
-  <collision>
-    <origin xyz="-0.465043 0.014202 -0.146068" rpy="0 0 0"/>
-    <geometry>
-      <mesh filename="package://RIVO_description/meshes/g_part_9_1.stl" scale="0.001 0.001 0.001"/>
-    </geometry>
-  </collision>
-</link>
-<link name="g_part_10_1">
-  <inertial>
-    <origin xyz="-0.014598965910585904 0.008272324580325768 8.800201478362246e-05" rpy="0 0 0"/>
-    <mass value="0.05700410540308428"/>
-    <inertia ixx="4e-06" iyy="3e-06" izz="6e-06" ixy="-0.0" iyz="-0.0" ixz="0.0"/>
-  </inertial>
-  <visual>
-    <origin xyz="-0.444042 0.006395 -0.132164" rpy="0 0 0"/>
-    <geometry>
-      <mesh filename="package://RIVO_description/meshes/g_part_10_1.stl" scale="0.001 0.001 0.001"/>
-    </geometry>
-    <material name="silver"/>
-  </visual>
-  <collision>
-    <origin xyz="-0.444042 0.006395 -0.132164" rpy="0 0 0"/>
-    <geometry>
-      <mesh filename="package://RIVO_description/meshes/g_part_10_1.stl" scale="0.001 0.001 0.001"/>
-    </geometry>
-  </collision>
-</link>
-<link name="g_part_1_1">
-  <inertial>
-    <origin xyz="0.036423386056162965 0.01149451999851355 0.006746851708180762" rpy="0 0 0"/>
-    <mass value="0.1054118615130382"/>
-    <inertia ixx="1.9e-05" iyy="4.8e-05" izz="5.5e-05" ixy="-1e-05" iyz="-3e-06" ixz="-9e-06"/>
-  </inertial>
-  <visual>
-    <origin xyz="-0.416441 0.014369 -0.132156" rpy="0 0 0"/>
-    <geometry>
-      <mesh filename="package://RIVO_description/meshes/g_part_1_1.stl" scale="0.001 0.001 0.001"/>
-    </geometry>
-    <material name="silver"/>
-  </visual>
-  <collision>
-    <origin xyz="-0.416441 0.014369 -0.132156" rpy="0 0 0"/>
-    <geometry>
-      <mesh filename="package://RIVO_description/meshes/g_part_1_1.stl" scale="0.001 0.001 0.001"/>
-    </geometry>
-  </collision>
-</link>
-<link name="g_part_6_1">
-  <inertial>
-    <origin xyz="0.010217406066357015 -0.0017233499857305518 0.004218909480987715" rpy="0 0 0"/>
-    <mass value="0.04741956072106952"/>
-    <inertia ixx="1e-06" iyy="1.9e-05" izz="2e-05" ixy="-3e-06" iyz="0.0" ixz="0.0"/>
-  </inertial>
-  <visual>
-    <origin xyz="-0.511072 0.022091 -0.137423" rpy="0 0 0"/>
-    <geometry>
-      <mesh filename="package://RIVO_description/meshes/g_part_6_1.stl" scale="0.001 0.001 0.001"/>
-    </geometry>
-    <material name="silver"/>
-  </visual>
-  <collision>
-    <origin xyz="-0.511072 0.022091 -0.137423" rpy="0 0 0"/>
-    <geometry>
-      <mesh filename="package://RIVO_description/meshes/g_part_6_1.stl" scale="0.001 0.001 0.001"/>
-    </geometry>
-  </collision>
-</link>
-<link name="g_part_7_1">
-  <inertial>
-    <origin xyz="0.011136128559519232 -0.006954489521749285 -0.005005307666391873" rpy="0 0 0"/>
-    <mass value="0.007386988595910908"/>
-    <inertia ixx="0.0" iyy="1e-06" izz="1e-06" ixy="0.0" iyz="-0.0" ixz="0.0"/>
-  </inertial>
-  <visual>
-    <origin xyz="-0.484818 0.005645 -0.141094" rpy="0 0 0"/>
-    <geometry>
-      <mesh filename="package://RIVO_description/meshes/g_part_7_1.stl" scale="0.001 0.001 0.001"/>
-    </geometry>
-    <material name="silver"/>
-  </visual>
-  <collision>
-    <origin xyz="-0.484818 0.005645 -0.141094" rpy="0 0 0"/>
-    <geometry>
-      <mesh filename="package://RIVO_description/meshes/g_part_7_1.stl" scale="0.001 0.001 0.001"/>
-    </geometry>
-  </collision>
-</link>
-<link name="g_part_3_1">
-  <inertial>
-    <origin xyz="-0.01973607073111644 -0.01515006847613011 0.002516844630100129" rpy="0 0 0"/>
-    <mass value="0.02397572621792568"/>
-    <inertia ixx="2e-06" iyy="2e-06" izz="4e-06" ixy="-1e-06" iyz="-0.0" ixz="0.0"/>
-  </inertial>
-  <visual>
-    <origin xyz="-0.489201 -0.031312 -0.146929" rpy="0 0 0"/>
-    <geometry>
-      <mesh filename="package://RIVO_description/meshes/g_part_3_1.stl" scale="0.001 0.001 0.001"/>
-    </geometry>
-    <material name="silver"/>
-  </visual>
-  <collision>
-    <origin xyz="-0.489201 -0.031312 -0.146929" rpy="0 0 0"/>
-    <geometry>
-      <mesh filename="package://RIVO_description/meshes/g_part_3_1.stl" scale="0.001 0.001 0.001"/>
-    </geometry>
-  </collision>
-</link>
-<link name="g_part_5_1">
-  <inertial>
-    <origin xyz="0.010187463177970035 0.0018070450955312463 -0.004255435248756628" rpy="0 0 0"/>
-    <mass value="0.0474195607210694"/>
-    <inertia ixx="1e-06" iyy="1.9e-05" izz="2e-05" ixy="3e-06" iyz="-0.0" ixz="0.0"/>
-  </inertial>
-  <visual>
-    <origin xyz="-0.509473 -0.022767 -0.146828" rpy="0 0 0"/>
-    <geometry>
-      <mesh filename="package://RIVO_description/meshes/g_part_5_1.stl" scale="0.001 0.001 0.001"/>
-    </geometry>
-    <material name="silver"/>
-  </visual>
-  <collision>
-    <origin xyz="-0.509473 -0.022767 -0.146828" rpy="0 0 0"/>
-    <geometry>
-      <mesh filename="package://RIVO_description/meshes/g_part_5_1.stl" scale="0.001 0.001 0.001"/>
-    </geometry>
-  </collision>
-</link>
-<link name="link_3_1">
-  <inertial>
-    <origin xyz="0.08880680552106898 0.006923559791520796 -0.001742253363287788" rpy="0 0 0"/>
-    <mass value="0.6955411833829301"/>
-    <inertia ixx="0.000129" iyy="0.003467" izz="0.003356" ixy="-5.6e-05" iyz="1e-06" ixz="-6e-06"/>
-  </inertial>
-  <visual>
-    <origin xyz="-0.014479 0.022897 -0.131606" rpy="0 0 0"/>
-    <geometry>
-      <mesh filename="package://RIVO_description/meshes/link_3_1.stl" scale="0.001 0.001 0.001"/>
-    </geometry>
-    <material name="silver"/>
-  </visual>
-  <collision>
-    <origin xyz="-0.014479 0.022897 -0.131606" rpy="0 0 0"/>
-    <geometry>
-      <mesh filename="package://RIVO_description/meshes/link_3_1.stl" scale="0.001 0.001 0.001"/>
-    </geometry>
-  </collision>
-</link>
-<joint name="dof_1" type="continuous">
-  <origin xyz="-3.5e-05 1.6e-05 0.091498" rpy="0 0 0"/>
-  <parent link="base_link"/>
-  <child link="link_2_1"/>
-  <axis xyz="2.3e-05 0.007455 -0.999972"/>
-</joint>
-<joint name="dof_2" type="continuous">
-  <origin xyz="0.014514 -0.022913 0.040108" rpy="0 0 0"/>
-  <parent link="link_2_1"/>
-  <child link="link_3_1"/>
-  <axis xyz="0.026148 -0.99963 -0.007452"/>
-</joint>
-<joint name="dof_3" type="continuous">
-  <origin xyz="0.217028 0.003698 -0.000463" rpy="0 0 0"/>
-  <parent link="link_3_1"/>
-  <child link="link_4_1"/>
-  <axis xyz="0.026148 -0.99963 -0.007452"/>
-</joint>
-<joint name="dof_4" type="continuous">
-  <origin xyz="0.184934 0.00483 0.001013" rpy="0 0 0"/>
-  <parent link="link_4_1"/>
-  <child link="g_part_1_1"/>
-  <axis xyz="-0.026148 0.99963 0.007452"/>
-</joint>
-<joint name="Rigid 6" type="fixed">
-  <origin xyz="0.068126 0.018679 0.014582" rpy="0 0 0"/>
-  <parent link="g_part_1_1"/>
-  <child link="g_part_12_1"/>
-</joint>
-<joint name="Rigid 9" type="fixed">
-  <origin xyz="0.068387 0.008683 0.014507" rpy="0 0 0"/>
-  <parent link="g_part_1_1"/>
-  <child link="g_part_4_1"/>
-</joint>
-<joint name="Rigid 10" type="fixed">
-  <origin xyz="0.068115 0.01872 0.009013" rpy="0 0 0"/>
-  <parent link="g_part_1_1"/>
-  <child link="g_part_8_1"/>
-</joint>
-<joint name="Rigid 13" type="fixed">
-  <origin xyz="0.048373 0.008334 0.004472" rpy="0 0 0"/>
-  <parent link="g_part_1_1"/>
-  <child link="g_part_2_1"/>
-</joint>
-<joint name="Rigid 14" type="fixed">
-  <origin xyz="0.048602 0.000167 0.013912" rpy="0 0 0"/>
-  <parent link="g_part_1_1"/>
-  <child link="g_part_9_1"/>
-</joint>
-<joint name="Rigid 16" type="fixed">
-  <origin xyz="0.027601 0.007974 8e-06" rpy="0 0 0"/>
-  <parent link="g_part_1_1"/>
-  <child link="g_part_10_1"/>
-</joint>
-<joint name="Rigid 18" type="fixed">
-  <origin xyz="0.026254 -0.016446 -0.003671" rpy="0 0 0"/>
-  <parent link="g_part_7_1"/>
-  <child link="g_part_6_1"/>
-</joint>
-<joint name="Rigid 19" type="fixed">
-  <origin xyz="0.068377 0.008724 0.008938" rpy="0 0 0"/>
-  <parent link="g_part_1_1"/>
-  <child link="g_part_7_1"/>
-</joint>
-<joint name="Rigid 21" type="fixed">
-  <origin xyz="-0.020272 0.008545 0.000101" rpy="0 0 0"/>
-  <parent link="g_part_5_1"/>
-  <child link="g_part_3_1"/>
-</joint>
-<joint name="Rigid 22" type="fixed">
-  <origin xyz="0.024906 0.018457 9e-05" rpy="0 0 0"/>
-  <parent link="g_part_12_1"/>
-  <child link="g_part_5_1"/>
-</joint>
-<transmission name="dof_1_trans">
-  <type>transmission_interface/SimpleTransmission</type>
-  <joint name="dof_1">
-    <hardwareInterface>hardware_interface/EffortJointInterface</hardwareInterface>
-  </joint>
-  <actuator name="dof_1_motor">
-    <hardwareInterface>hardware_interface/EffortJointInterface</hardwareInterface>
-    <mechanicalReduction>1</mechanicalReduction>
-  </actuator>
-</transmission>
-<transmission name="dof_2_trans">
-  <type>transmission_interface/SimpleTransmission</type>
-  <joint name="dof_2">
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
Commit message: muthal machine ready

File: RIVO_description/urdf/RIVO.xacro (robot description, xacro)
@@ -14,6 +14,6 @@
     <inertial>
       <origin xyz="0.002894864480150963 0.0004061893631920555 0.029121311645850093" rpy="0 0 0"/>
-      <mass value="2.3408931898157137"/>
-      <inertia ixx="0.004521" iyy="0.004886" izz="0.00607" ixy="4e-06" iyz="-9e-06" ixz="5.9e-05"/>
+      <mass value="100.3408931898157137"/>
+      <inertia ixx="0.4521" iyy="0.4886" izz="0.607" ixy="4e-04" iyz="-9e-04" ixz="5.9e-03"/>
     </inertial>
     <visual>

Commit message: add inverseK

File: RIVO_description/urdf/RIVO.xacro (robot description, xacro)
@@ -15,5 +15,5 @@
       <origin xyz="0.002894864480150963 0.0004061893631920555 0.029121311645850093" rpy="0 0 0"/>
       <mass value="100.3408931898157137"/>
-      <inertia ixx="0.4521" iyy="0.4886" izz="0.607" ixy="4e-04" iyz="-9e-04" ixz="5.9e-03"/>
+      <inertia ixx="45.21" iyy="48.86" izz="60.7" ixy="4e-02" iyz="-9e-02" ixz="5.9e-01"/>
     </inertial>
     <visual>
@@ -316,5 +316,5 @@
     <child link="link_2_1"/>
     <axis xyz="2.3e-05 0.007455 -0.999972"/>
-    <limit lower="0" upper="3.142" effort="300" velocity="3"/>
+    <limit lower="-1.57" upper="1.57" effort="300" velocity="3"/>
   </joint>
   <joint name="dof_2" type="revolute">
@@ -323,5 +323,5 @@
     <child link="link_3_1"/>
     <axis xyz="0.026148 -0.99963 -0.007452"/>
-    <limit lower="0" upper="3.142" effort="300" velocity="3"/>
+    <limit lower="-1.57" upper="1.57" effort="300" velocity="3"/>
   </joint>
   <joint name="dof_3" type="revolute">
@@ -330,5 +330,5 @@
     <child link="link_4_1"/>
     <axis xyz="0.026148 -0.99963 -0.007452"/>
-    <limit lower="0" upper="3.142" effort="300" velocity="3"/>
+    <limit lower="-3.142" upper="0" effort="300" velocity="3"/>
   </joint>
   <joint name="dof_4" type="revolute">
@@ -336,6 +336,6 @@
     <parent link="link_4_1"/>
     <child link="g_part_1_1"/>
-    <axis xyz="-0.026148 0.99963 0.007452"/>
-    <limit lower="0" upper="3.142" effort="300" velocity="3"/>
+    <axis xyz="0.026148 -0.99963 -0.007452"/>
+    <limit lower="-3.142" upper="3.142" effort="300" velocity="3"/>
   </joint>
   <joint name="Rigid 6" type="fixed">
